File: pcb/pcb.kicad_pcb (KiCad board)
At the start: 2 copper layers, 229.9 x 97.8 mm, 154 parts, among them J1 USB_C_Receptacle_USB2.0, SW1 Reset, SW10 SW_Push, SW11 SW_Push, SW12 SW_Push, SW13 SW_Push, SW14 SW_Push, SW15 SW_Push, SW16 SW_Push, SW17 SW_Push, SW18 SW_Push, SW19 SW_Push, SW2 SW_Push, SW20 SW_Push, SW21 SW_Push, SW22 SW_Push, SW23 SW_Push, SW24 SW_Push, SW25 SW_Push, SW26 SW_Push, SW27 SW_Push, SW28 SW_Push, SW29 SW_Push, SW3 SW_Push, SW30 SW_Push, SW31 SW_Push, SW32 SW_Push, SW33 SW_Push, SW34 SW_Push, SW35 SW_Push, SW36 SW_Push, SW37 SW_Push, SW38 SW_Push, SW39 SW_Push, SW4 SW_Push, SW40 SW_Push, SW41 SW_Push, SW42 SW_Push, SW43 SW_Push, SW44 SW_Push, SW45 SW_Push, SW46 SW_Push, SW47 SW_Push, SW48 SW_Push, SW49 SW_Push, SW5 SW_Push, SW50 SW_Push, SW51 SW_Push, SW52 SW_Push, SW53 SW_Push, SW54 SW_Push, SW55 SW_Push, SW56 SW_Push, SW57 SW_Push, SW58 SW_Push, SW59 SW_Push, SW6 SW_Push, SW60 SW_Push, SW7 SW_Push, SW8 SW_Push, SW9 SW_Push, U1 ATmega32U4-AU, Y1 TSX3225

Commit message: Add name and author to PCB
Other:
- board text added: "Designed by Maxr1998"
- board text added: "Phoebe Keyboard"
- board text added: "·"
Changed lines of the file:
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@@
   (general
     (thickness 1.6)
-    (drawings 21)
+    (drawings 24)
     (tracks 1131)
     (zones 0)
@@
     )
   )
+  (gr_text · (at 240.03 124.46) (layer B.SilkS)
+    (effects (font (size 1 1) (thickness 0.15)) (justify mirror))
+  )
+  (gr_text "Designed by Maxr1998" (at 230.505 124.46) (layer B.SilkS)
+    (effects (font (size 1 1) (thickness 0.15)) (justify mirror))
+  )
+  (gr_text "Phoebe Keyboard" (at 247.65 124.46) (layer B.SilkS)
+    (effects (font (size 1 1) (thickness 0.15)) (justify mirror))
+  )
   (gr_line (start 133.35 96.52) (end 133.35 115.57) (layer Dwgs.User) (width 0.15))

Commit message: Add infill, reroute col11
Routing:
- net col11: track 210.5 -> 184.8 mm
- added copper zone on B.Cu, net GND
- added copper zone on F.Cu, net GND
